Commit message: SImulation of a spider robot using reinforcement learning.

File: spiderbot_assy/spiderbot_assy.urdf (robot description, URDF)
Before this commit: robot spiderbot_assy, 9 links, 8 joints
Joints:
- removed joint base_link_Revolute-2
- removed joint base_link_Revolute-4
- removed joint knee_FL_Revolute-6
- removed joint knee_FR_Revolute-7
- removed joint knee_RL_Revolute-10
- added joint base_link_Revolute-1: type revolute, parent base_link, child knee_FL, origin xyz=0.08911 0.062000000000000006 0.01835 rpy=3.141592653589793 -0.0 0.0, axis 0.0 0.0 1.0, limit lower=-0.087266 upper=1.308997 effort=1000000 velocity=1000000
- added joint base_link_Revolute-7: type revolute, parent base_link, child knee_RR, origin xyz=-0.08911 -0.062000000000000006 0.01835 rpy=-3.141592653589783 -0.0 0.0, axis 0.0 1.04744440165294e-14 1.0, limit lower=-0.087266 upper=1.308997 effort=1000000 velocity=1000000
- added joint knee_FL_Revolute-2: type revolute, parent knee_FL, child leg_FL, origin xyz=0.01835000000000001 -0.032 0.03011 rpy=-3.141592653589776 1.5707963267948966 0, axis -1.232595164407831e-32 1.7457406694215667e-14 1.0, limit lower=-0.523599 upper=1.919862 effort=1000000 velocity=1000000
- added joint knee_FR_Revolute-4: type revolute, parent knee_FR, child leg_FR, origin xyz=0.01785 0.032 0.03011 rpy=1.7457406694215667e-14 1.5707963267948966 0, axis 0.0 -1.7457406694215667e-14 -1.0, limit lower=-1.919862 upper=0.523599 effort=1000000 velocity=1000000
- added joint knee_RL_Revolute-6: type revolute, parent knee_RL, child leg_RL, origin xyz=0.018497009999999998 -0.03191524999999999 0.03011 rpy=-3.141592653589776 1.5707963267948966 0, axis 0.0 0.004600000000017457 0.9999889999999999, limit lower=-0.436332 upper=1.919862 effort=1000000 velocity=1000000
- joint base_link_Revolute-3: axis 0.0 4.4520966792844554e-18 1.0 -> -0.0 -7.782894391141709e-17 1.0; child knee_RL -> knee_FR; limit lower=-1.308997 upper=0.087266 effort=1000000 velocity=1000000 -> lower=1.832596 upper=3.403392 effort=1000000 velocity=1000000; origin xyz=-0.08911 0.062000000000000006 0.01835 rpy=-3.141592653589793 -0.0 0.0 -> xyz=0.08911 -0.062000000000000006 0.01835 rpy=3.141592653589793 -0.0 0.0
- joint base_link_Revolute-5: axis -0.0 -7.782894391141709e-17 1.0 -> 0.0 4.4520966792844554e-18 1.0; child knee_FR -> knee_RL; limit lower=-4.45059 upper=-3.054326 effort=1000000 velocity=1000000 -> lower=-1.308997 upper=0.087266 effort=1000000 velocity=1000000; origin xyz=0.08911 -0.062000000000000006 0.01835 rpy=3.141592653589793 -0.0 0.0 -> xyz=-0.08911 0.062000000000000006 0.01835 rpy=-3.141592653589793 -0.0 0.0
